File: Breakout/AFE/MAX30003/MAX30003.kicad_pcb (KiCad board)
At the start: 2 copper layers, 16 parts, among them IC1 MAX30003CTI+, J1 Conn_01x02_Male, J2 Conn_01x06, J3 Conn_01x04, X1 KX2013E0032.768000

Commit message: qdone
Parts:
- removed the J1 at (239.7, 87.1)
- removed the J3 at (235.2, 75.4)
- added J1: Conn_01x02_Male, Connector_PinHeader_2.54mm:PinHeader_1x02_P2.54mm_Vertical, F.Cu at (130.8, 86.3)
- added J1: Conn_01x09, Connector_PinHeader_2.54mm:PinHeader_1x09_P2.54mm_Vertical, F.Cu at (130.9, 103.8)
- added J3: Conn_01x04, Connector_PinHeader_2.54mm:PinHeader_1x04_P2.54mm_Vertical, F.Cu at (130.8, 92.5)
- added J3: Conn_01x02, Connector_PinHeader_2.54mm:PinHeader_1x02_P2.54mm_Vertical, F.Cu at (148.5, 78.4)
- C1, C2, C6, C8: footprint Capacitor_SMD:C_0603_1608Metric -> Capacitor_SMD:C_0805_2012Metric
- J2: footprint Connector_PinHeader_2.54mm:PinHeader_1x06_P2.54mm_Vertical -> Connector_PinHeader_2.54mm:PinHeader_1x11_P2.54mm_Vertical
- moved C3 102.4 mm to (137.6, 83.2)
- moved C10 101.5 mm to (137.9, 94.4)
- moved C11 101.5 mm to (139.4, 94.4)
- moved C1 101.2 mm to (140.3, 83.4)
- moved C8 101.1 mm to (141.4, 95.4)
- moved C9 100.7 mm to (143.3, 94.4)
- moved IC1 100.7 mm to (141.2, 89.3)
- moved X1 100.7 mm to (145.7, 92.9)
- moved C5 100.7 mm to (145.1, 95.6)
- moved C2 100.5 mm to (142.6, 83.4)
- moved C7 100.4 mm to (146.9, 95.6)
- moved C4 99.7 mm to (145.7, 82.8)
- moved C6 99.7 mm to (145.8, 84.8)
- moved J2 97.0 mm to (154.8, 103.8)
Connections:
- net /CSB renamed /MAX30003_CSB
- net /INT2B renamed /MAX30003_INT2B
- net /INTB renamed /MAX30003_INTB
- net /SCLK renamed /MAX30003_SCLK
- net /SDI renamed /MAX30003_SDI
- net /SDO renamed /MAX30003_SDO
- IC1 pad 19: DVDD -> AVDD
Routing:
- net AVDD: track 5.39 -> 35.9 mm, vias 0 -> 3
- net DGND: track 39.7 -> 68.4 mm
- net /MAX30003_SCLK: track 6.35 -> 19.1 mm
- net /MAX30003_SDI: track 6.27 -> 18.2 mm
- net /MAX30003_CSB: track 8.63 -> 20.0 mm
- net AGND: track 25.8 -> 15.1 mm, vias 0 -> 1
- net /MAX30003_SDO: track 7.12 -> 16.1 mm
- net /MAX30003_INT2B: track 9.15 -> 15.4 mm
- net /MAX30003_INTB: track 10.8 -> 14.0 mm
- net DVDD: track 25.7 -> 28.3 mm
- net Net-(C3-Pad1): track 2.23 -> 4.26 mm
- net Net-(C10-Pad2): track 5.44 -> 6.75 mm
- net Net-(C11-Pad1): track 2.41 -> 3.56 mm
- net Net-(C10-Pad1): track 3.09 -> 4.22 mm
- net /SWDIO: track 0.00 -> 1.05 mm
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- added copper zone on B.Cu, net AGND
- added copper zone on F.Cu, net AGND
Other:
- board outline added: 30 x 30.4 mm
- net class 6 added: clearance 0.1524, trace_width 0.1524, via_dia 0.7, via_drill 0.6
- net class Default: trace_width 0.152 -> 0.2032; via_dia 0.508 -> 0.7; via_drill 0.3302 -> 0.6
- rule trace_min: 0.05 -> 0.0508
- rule via_min_drill: 0.3302 -> 0.3
- rule via_min_size: 0.152 -> 0.4
