File: Breakout/AFE/MAX30003/MAX30003.sch (KiCad schematic (older format))
At the start: 16 parts, among them IC1 MAX30003CTI+, J1 Conn_01x02_Male, J2 Conn_01x06, J3 Conn_01x04, X1 KX2013E0032.768000

Commit message: qdone
Parts:
- C1, C2, C6, C8: footprint Capacitor_SMD:C_0603_1608Metric -> Capacitor_SMD:C_0805_2012Metric
- J2: footprint Connector_PinHeader_2.54mm:PinHeader_1x06_P2.54mm_Vertical -> Connector_PinHeader_2.54mm:PinHeader_1x11_P2.54mm_Vertical
Connections:
- net AVDD: now also IC1.19 (OVDD)
- net DVDD: no longer IC1.19 (OVDD)
- net CSB renamed MAX30003_CSB
- net INT2B renamed MAX30003_INT2B
- net INTB renamed MAX30003_INTB
- net SCLK renamed MAX30003_SCLK
- net SDI renamed MAX30003_SDI
- net SDO renamed MAX30003_SDO
- no-connect marks 0 -> 1
Changed lines of the file:
@@
 F 0 "C2" H 3150 1000 40  0000 L CNN
 F 1 "10uF" H 3156 815 40  0000 L CNN
-F 2 "Capacitor_SMD:C_0603_1608Metric" H 3188 750 30  0001 C CNN
+F 2 "Capacitor_SMD:C_0805_2012Metric" H 3188 750 30  0001 C CNN
 F 3 "~" H 3150 900 60  0000 C CNN
 	1    3150 900
@@
 F 0 "C1" H 2700 1000 40  0000 L CNN
 F 1 "10uF" H 2706 815 40  0000 L CNN
-F 2 "Capacitor_SMD:C_0603_1608Metric" H 2738 750 30  0001 C CNN
+F 2 "Capacitor_SMD:C_0805_2012Metric" H 2738 750 30  0001 C CNN
 F 3 "~" H 2700 900 60  0000 C CNN
 	1    2700 900
@@
 AVDD
 Text GLabel 4750 2950 2    50   Input ~ 0
-DVDD
+AVDD
 $Comp
 L Device:C C10
@@
 F 0 "C8" H 4550 4050 40  0000 L CNN
 F 1 "10uF" H 4556 3865 40  0000 L CNN
-F 2 "Capacitor_SMD:C_0603_1608Metric" H 4588 3800 30  0001 C CNN
+F 2 "Capacitor_SMD:C_0805_2012Metric" H 4588 3800 30  0001 C CNN
 F 3 "~" H 4550 3950 60  0000 C CNN
 	1    4550 3950
@@
 F 0 "C6" H 3900 1800 40  0000 L CNN
 F 1 "10uF" H 4056 1615 40  0000 L CNN
-F 2 "Capacitor_SMD:C_0603_1608Metric" H 4088 1550 30  0001 C CNN
+F 2 "Capacitor_SMD:C_0805_2012Metric" H 4088 1550 30  0001 C CNN
 F 3 "~" H 4050 1700 60  0000 C CNN
 	1    4050 1700
@@
 DGND
 Text Label 4750 2750 0    50   ~ 0
-INTB
+MAX30003_INTB
 Text Label 4750 2850 0    50   ~ 0
-INT2B
+MAX30003_INT2B
 Text Label 5000 3050 0    50   ~ 0
-SDO
+MAX30003_SDO
 Wire Wire Line
 	4150 3050 5000 3050
 Text Label 5000 3150 0    50   ~ 0
-SDI
+MAX30003_SDI
 Text Label 5000 3250 0    50   ~ 0
-SCLK
+MAX30003_SCLK
 Text Label 5000 3350 0    50   ~ 0
-CSB
+MAX30003_CSB
 Wire Wire Line
 	4150 3150 5000 3150
@@
 Wire Wire Line
 	4150 3350 5000 3350
-Text Label 6300 2950 0    50   ~ 0
-INTB
 Wire Wire Line
 	5900 2950 6300 2950
-Text Label 6300 3050 0    50   ~ 0
-INT2B
 Wire Wire Line
 	6300 3050 5900 3050
-Text Label 6300 3150 0    50   ~ 0
-SDO
 Wire Wire Line
 	6300 3150 5900 3150
-Text Label 6300 3250 0    50   ~ 0
-SDI
-Text Label 6300 3350 0    50   ~ 0
-SCLK
-Text Label 6300 3450 0    50   ~ 0
-CSB
 Wire Wire Line
 	5900 3250 6300 3250
@@
 F 0 "J2" H 5620 2725 50  0000 C CNN
 F 1 "Conn_01x06" H 5620 2816 50  0000 C CNN
-F 2 "Connector_PinHeader_2.54mm:PinHeader_1x06_P2.54mm_Vertical" H 5700 3250 50  0001 C CNN
+F 2 "Connector_PinHeader_2.54mm:PinHeader_1x11_P2.54mm_Vertical" H 5700 3250 50  0001 C CNN
 F 3 "~" H 5700 3250 50  0001 C CNN
 	1    5700 3250
 	-1   0    0    1
 $EndComp
+Text Label 6300 2950 0    50   ~ 0
+MAX30003_INTB
+Text Label 6300 3050 0    50   ~ 0
+MAX30003_INT2B
+Text Label 6300 3150 0    50   ~ 0
+MAX30003_SDO
+Text Label 6300 3250 0    50   ~ 0
+MAX30003_SDI
+Text Label 6300 3350 0    50   ~ 0
+MAX30003_SCLK
+Text Label 6300 3450 0    50   ~ 0
+MAX30003_CSB
+NoConn ~ 5300 1400
 $EndSCHEMATC
