File: Breakout/IMU/BMI160/BMI160_Breakout/BMI160_Breakout.kicad_pcb (KiCad board)
At the start: 2 copper layers, 20 x 20 mm, 7 parts, among them J1 I2C, J2 Power, U1 BMI160

Commit message: qdone
Parts:
- removed J1: I2C, Connector_PinHeader_2.54mm:PinHeader_1x05_P2.54mm_Vertical
- removed the J2 at (144.2, 65.5)
- added J2: Conn_01x04, Connector_PinHeader_2.54mm:PinHeader_1x04_P2.54mm_Vertical, F.Cu at (186.0, 94.0)
- added J2: Conn_01x11, Connector_PinHeader_2.54mm:PinHeader_1x11_P2.54mm_Vertical, F.Cu at (210.0, 97.7)
- added J3: Conn_01x02, Connector_PinHeader_2.54mm:PinHeader_1x02_P2.54mm_Vertical, F.Cu at (203.7, 72.3)
- added J3: Conn_01x09, Connector_PinHeader_2.54mm:PinHeader_1x09_P2.54mm_Vertical, F.Cu at (186.1, 97.7)
- moved R1 65.0 mm to (197.0, 78.5)
- moved R2 63.7 mm to (199.0, 78.5), turned to 90 degrees
- moved U1 63.4 mm to (198.4, 82.7)
- moved C1 63.4 mm to (202.2, 85.2)
- moved C2 62.4 mm to (197.6, 85.4)
Connections:
- C1 pad 1: VDD-Vin -> AVDD
- C1 pad 2: DGND -> AGND
- C2 pad 1: GNDIO -> DGND
- C2 pad 2: VDDIO-Vin -> DVDD
- R1 pad 2: VDDIO-Vin -> DVDD
- R2 pad 2: VDDIO-Vin -> DVDD
- U1 pad 1: (no net) -> DGND
- U1 pad 10: (no net) -> Net-(U1-Pad10)
- U1 pad 11: (no net) -> Net-(U1-Pad11)
- U1 pad 12: (no net) -> DVDD
- U1 pad 13: (no net) -> /BMI_SCL
- U1 pad 14: (no net) -> /BMI_SDA
- U1 pad 2: (no net) -> Net-(U1-Pad2)
- U1 pad 3: (no net) -> Net-(U1-Pad3)
- U1 pad 4: (no net) -> /BMI_INT1
- U1 pad 5: (no net) -> DVDD
- U1 pad 6: (no net) -> DGND
- U1 pad 7: (no net) -> AGND
- U1 pad 8: (no net) -> AVDD
- U1 pad 9: (no net) -> /BMI_INT2
Routing:
- net DVDD: track 0.00 -> 34.6 mm, vias 0 -> 2
- net AVDD: track 0.00 -> 22.8 mm
- net GNDIO: track 22.5 -> 0.00 mm
- net AGND: track 0.00 -> 20.7 mm
- net VDDIO-Vin: track 20.7 -> 0.00 mm
- net /BMI_INT2: track 28.2 -> 11.7 mm
- net /BMI_SDA: track 7.74 -> 19.4 mm, vias 0 -> 1
- net /BMI_INT1: track 7.60 -> 18.5 mm, vias 0 -> 1
- net DGND: track 14.6 -> 4.68 mm, vias 0 -> 2
- net VDD-Vin: track 8.13 -> 0.00 mm
- net /BMI_SA0: track 7.05 -> 0.00 mm
- net /BMI_SCL: track 9.78 -> 16.7 mm
- added copper zone on B.Cu, net DGND
- added copper zone on F.Cu, net DGND
Other:
- board size 20 x 20 mm -> 30 x 30.4 mm
- net class 6 added: clearance 0.1524, trace_width 0.1524, via_dia 0.7, via_drill 0.6
- net class Default: trace_width 0.4572 -> 0.2032; via_dia 0.508 -> 0.7; via_drill 0.3302 -> 0.6
- rule trace_min: 0.2 -> 0.0508
