File: Breakout/IMU/BMI160/BMI160_Breakout/BMI160_Breakout.sch (KiCad schematic (older format))
At the start: 7 parts, among them J1 Conn_01x05, J2 Conn_01x04, U1 BMI160

Commit message: qdone
Parts:
- removed J1: Conn_01x05, Connector_PinHeader_2.54mm:PinHeader_1x05_P2.54mm_Vertical, symbol Connector_Generic:Conn_01x05
- added J1: Conn_01x11, symbol Connector_Generic:Conn_01x11
Connections:
- net BMI_SA0 is gone; now on net DGND: U1.1 (SDO)
- net BMI_INT1: now also J1.9 (Pin_9)
- net BMI_INT2: now also J1.8 (Pin_8)
- net BMI_SCL: now also J1.11 (Pin_11)
- net BMI_SDA: now also J1.10 (Pin_10)
- net DGND: now also C2.1, J2.2 (Pin_2), U1.6 (GNDIO); no longer C1.2, J2.3 (Pin_3), U1.7 (GND)
- removed net GNDIO: C2.1, J2.1 (Pin_1), U1.6 (GNDIO)
- net VDD-Vin renamed AVDD
- net AVDD: now also J2.3 (Pin_3); no longer J2.4 (Pin_4)
- net VDDIO-Vin renamed DVDD
- net DVDD: now also J2.1 (Pin_1); no longer J2.2 (Pin_2)
- new net AGND: C1.2, J2.4 (Pin_4), U1.7 (GND)
Changed lines of the file:
@@
 EESchema Schematic File Version 4
+LIBS:BMI160_Breakout-cache
 EELAYER 26 0
 EELAYER END
@@
 	0    1    1    0
 $EndComp
-Text GLabel 3500 3550 3    60   Input ~ 0
-GNDIO
 NoConn ~ -6050 -2500
 NoConn ~ 11600 -1550
@@
 Text Label 4000 2600 0    50   ~ 0
 BMI_INT2
-Text Label 2700 2200 3    50   ~ 0
-BMI_SA0
 Text Label 2650 2800 3    50   ~ 0
 BMI_INT1
 Text Notes 5000 2850 0    50   ~ 0
 SDO: Address Select I2C\nASD: Magneto Interface (not used)\nASC: Magneto Interface (Not used)\nINT1, INT2: Interrupt Pin\nVDDIO: 1.2V-3.6V\nGNDIO: Ground IO\nGND: Ground IO/Analog\nVDD: Analog Power (1.7V-3.6V)\nOCSB. OSDP: OIS Interface (not used)\nCSB: Chip Select for SPI/Protocol Selection Pin\nSCx: SCL I2C. Serial Clock\nSDx: SDA I2C\n
-Text GLabel 2350 3550 0    50   Input ~ 0
-VDDIO-Vin
 $Comp
 L Device:C C2
@@
 Wire Wire Line
 	3750 3200 3750 3550
-Text GLabel 3750 3550 3    60   Input ~ 0
-DGND
-Text GLabel 4300 3200 3    50   Input ~ 0
-VDD-Vin
-$Comp
-L Connector_Generic:Conn_01x05 J1
-U 1 1 5D75DA3A
-P 7400 1400
-F 0 "J1" H 7320 975 50  0000 C CNN
-F 1 "Conn_01x05" H 7320 1066 50  0000 C CNN
-F 2 "Connector_PinHeader_2.54mm:PinHeader_1x05_P2.54mm_Vertical" H 7400 1400 50  0001 C CNN
-F 3 "~" H 7400 1400 50  0001 C CNN
-	1    7400 1400
-	-1   0    0    1
-$EndComp
-Text Label 8100 1400 0    50   ~ 0
+Text Label 9600 1150 0    50   ~ 0
 BMI_SDA
-Wire Wire Line
-	7600 1200 8100 1200
-Text Label 8100 1500 0    50   ~ 0
+Text Label 9600 1050 0    50   ~ 0
 BMI_SCL
-Wire Wire Line
-	7600 1300 8100 1300
-Text Label 8100 1600 0    50   ~ 0
+Text Label 9600 1350 0    50   ~ 0
 BMI_INT2
-Wire Wire Line
-	7600 1600 8100 1600
-Text Label 8100 1300 0    50   ~ 0
-BMI_SA0
-Text Label 8100 1200 0    50   ~ 0
+Text Label 9600 1250 0    50   ~ 0
 BMI_INT1
-Wire Wire Line
-	7600 1400 8100 1400
-Wire Wire Line
-	8100 1500 7600 1500
 $Comp
 L Connector_Generic:Conn_01x04 J2
@@
 	-1   0    0    1
 $EndComp
-Text GLabel 8100 1850 2    50   Input ~ 0
-VDD-Vin
+Text GLabel 8100 1950 2    50   Input ~ 0
+AVDD
 Wire Wire Line
 	8100 1850 7600 1850
-Text GLabel 8100 1950 2    60   Input ~ 0
+Text GLabel 8100 1850 2    60   Input ~ 0
+AGND
+Wire Wire Line
+	8100 1950 7600 1950
+Text GLabel 8100 2050 2    60   Input ~ 0
 DGND
-Wire Wire Line
-	8100 1950 7600 1950
-Text GLabel 8100 2150 2    60   Input ~ 0
-GNDIO
-Text GLabel 8100 2050 2    50   Input ~ 0
-VDDIO-Vin
+Text GLabel 8100 2150 2    50   Input ~ 0
+DVDD
 Wire Wire Line
 	8100 2050 7600 2050
 Wire Wire Line
 	8100 2150 7600 2150
+Text GLabel 2700 2200 0    60   Input ~ 0
+DGND
+$Comp
+L Connector_Generic:Conn_01x11 J1
+U 1 1 5D8F871F
+P 9400 1550
+F 0 "J1" H 9320 825 50  0000 C CNN
+F 1 "Conn_01x11" H 9320 916 50  0000 C CNN
+F 2 "" H 9400 1550 50  0001 C CNN
+F 3 "~" H 9400 1550 50  0001 C CNN
+	1    9400 1550
+	-1   0    0    1
+$EndComp
+Text GLabel 4300 3400 3    60   Input ~ 0
+AVDD
+Wire Wire Line
+	4300 3200 4300 3400
+Connection ~ 4300 3200
+Text GLabel 3500 3550 3    60   Input ~ 0
+DGND
+Text GLabel 3750 3550 3    60   Input ~ 0
+AGND
+Text GLabel 2350 3550 0    50   Input ~ 0
+DVDD
 $EndSCHEMATC
